File: KiCad/Clock.sch (KiCad schematic (older format))
At the start: 9 parts, among them U1 NE555

Commit message: Added clock mode toggle logic
Parts:
- added C?: 100nF, symbol C
- added C? (x3): 10nF, symbol C
- added D? (x3): LED, symbol LED
- added R? (x5): 1K, symbol R
- added R?: 1M, symbol R
- added R? (x3): 330, symbol R
- added SW1: SW_SPST, symbol SW_SPST
- added SW? (x2): SW_DPDT_x2, symbol SW_DPDT_x2
- added U? (x3): NE555, symbol NE555
- added U? (x7): 74LS08, symbol 74LS08
- added U? (x3): 74LS32, symbol 74LS32
- added U? (x3): 74LS04, symbol 74LS04
- added Y?: 1 MHz, symbol Crystal_GND2
- R1: value 220 -> 330
Connections:
- net labels added: CLK_HLT, CLK_MAN, CLK_MAN_EN, CLK_TURBO, CLK_TURBO_EN, CLOCK
- wire segments 43 -> 192
Other:
- note added: "Clock mode toggle logic"
- note added: "Manual (single-step) clock"
- note added: "Manual (single-step) clock toggle switch"
- note added: "Turbo clock (1 MHz)"
- note added: "Turbo clock toggle switch"

Commit message: First revision of Clock module circuit (untested at this point)
Parts:
- removed SW1: SW_SPST, symbol SW_SPST
- removed SW? (x2): SW_DPDT_x2, symbol SW_DPDT_x2
- added SW1: SW_Push, symbol SW_Push
- added SW2, SW3: SW_Push_SPDT, symbol SW_Push_SPDT
- gave numbers to parts that had none: 24
Connections:
- net labels added: VCC
- wire segments 192 -> 151
- no-connect marks 0 -> 4
