File: Circuits/KiCad/Main-Board/Main-Board.kicad_pcb (KiCad board)
At the start: 2 copper layers, 284.5 x 484.5 mm, 58 parts, among them J1 CLOCK, J10 ALU_0, J11 ALU_1, J12 IR_0, J13 MAR_0, J14 PROGRAM-COUNTER_1, J15 IR_1, J16 SP_0, J17 MAR_1_ADDRESS-IN, J18 SP_1_MEMORY-ADDRESS, J19 MAR_2_ADDRESS-OUT, J2 MEMORY_0, J20 CONTROLLER_0, J21 CONTROLLER_1, J22 CONTROLLER_2, J23 Barrel_Jack, J24 CLOCK_1, J25 CLOCK_2, J26 CLOCK_3, J27 FLAGS-REGISTER_1, J28 FLAGS-REGISTER_2, J29 MEMORY_2, J3 REGISTER-A, J30 MEMORY_3, J31 MAR_3, J32 REGISTER-A_1, J33 REGISTER-A_2, J34 REGISTER-C_1, J35 REGISTER-C_2, J36 REGISTER-B_1, J37 REGISTER-B_2, J38 REGISTER-D_1, J39 REGISTER-D_2, J4 REGISTER-C, J5 FLAGS-REGISTER, J6 MEMORY_1, J7 REGISTER-B, J8 REGISTER-D, J9 PROGRAM-COUNTER_0, SW1 SW_Push_SPDT, U1 74x04

Commit message: Removed old (obsolete) circuit schematics
Parts:
- moved J20 1.14 mm to (169.7, 419.1)
- moved C15 1.14 mm to (166.5, 419.1)
- moved J21 1.14 mm to (322.1, 457.2)
- moved J22 0.76 mm to (327.2, 515.6)
Other:
- board size 284.5 x 484.5 mm -> 286.4 x 484.5 mm

Commit message: Rerouted Controller and Main board (needs work)
Routing:
- net +5V: track 0.00 -> 1010.9 mm
- net GND: track 0.00 -> 996.8 mm
- net CLOCK: track 0.00 -> 915.4 mm, vias 0 -> 1
- net DATA_BUS1: track 0.00 -> 722.6 mm
- net DATA_BUS2: track 0.00 -> 722.2 mm
- net DATA_BUS6: track 0.00 -> 722.1 mm
- net DATA_BUS4: track 0.00 -> 721.8 mm
- net DATA_BUS0: track 0.00 -> 720.6 mm
- net DATA_BUS5: track 0.00 -> 720.2 mm
- net DATA_BUS7: track 0.00 -> 719.6 mm
- net DATA_BUS3: track 0.00 -> 710.8 mm
- net Fc_out: track 0.00 -> 556.1 mm, vias 0 -> 1
- net ~PC_MAR_out: track 0.00 -> 547.0 mm, vias 0 -> 1
- net ~STK_MAR_out: track 0.00 -> 512.3 mm, vias 0 -> 2
- net ~ALU_AY_load: track 0.00 -> 490.6 mm
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
Commit message: Finished Main Board PCB
Routing:
- net GND: track 996.8 -> 217.2 mm
- net +5V: track 1010.9 -> 1013.5 mm
- net DATA_BUS5: track 720.2 -> 717.7 mm
- net DATA_BUS6: track 722.1 -> 720.0 mm
- net CLOCK: track 915.4 -> 913.6 mm
- net DATA_BUS2: track 722.2 -> 720.5 mm
- net DATA_BUS3: track 710.8 -> 709.1 mm
- net DATA_BUS4: track 721.8 -> 720.3 mm
- net DATA_BUS1: track 722.6 -> 721.1 mm
- net DATA_BUS7: track 719.6 -> 718.3 mm
- net A4: track 257.4 -> 256.2 mm
- net A1: track 259.0 -> 258.1 mm
- net A8: track 256.9 -> 256.0 mm
- net DATA_BUS0: track 720.6 -> 719.7 mm
- net A12: track 256.8 -> 256.0 mm
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- added copper zone on B.Cu, net GND

Commit message: Last PCB's put into production
Other:
- board text added: "REVISION 1 - 2019/08/16 https://github.com/DutchMaker/TTL-Computer"
- board text added: "↓ ARITHMETIC LOGIC UNIT ↓"
- board text added: "↓ CLOCK ↓"
- board text added: "↓ CONTROLLER ↓"
- board text added: "↓ FLAGS ↓"
- board text added: "↓ INSTRUCTION ↓"
- board text added: "↓ MEMORY ACCESS REGISTER ↓"
- board text added: "↓ MEMORY ↓"
- board text added: "↓ PROGRAM COUNTER ↓"
- board text added: "↓ REGISTER A ↓"
- board text added: "↓ REGISTER B ↓"
- board text added: "↓ REGISTER C ↓"
- board text added: "↓ REGISTER D ↓"
- board text added: "↓ STACK POINTER ↓"
- board text removed: "ARITHMETIC LOGIC UNIT"
- board text removed: "CONTROLLER"
- board text removed: "FLAGS REGISTER"
- board text removed: "INSTRUCTION REGISTER"
- board text removed: "MEMORY"
- board text removed: "MEMORY ACCESS REGISTER"
- board text removed: "PROGRAM COUNTER"
- board text removed: "REGISTER A"
- board text removed: "REGISTER B"
- board text removed: "REGISTER C"
- board text removed: "REGISTER D"
- board text removed: "STACK POINTER"
Changed lines of the file:
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@@
-(kicad_pcb (version 20171130) (host pcbnew 5.0.2+dfsg1-1)
+(kicad_pcb (version 20171130) (host pcbnew "(5.1.2)-2")
   (general
     (thickness 1.6)
-    (drawings 402)
+    (drawings 390)
     (tracks 1197)
     (zones 0)
@@
     (34 B.Paste user hide)
     (35 F.Paste user hide)
-    (36 B.SilkS user hide)
+    (36 B.SilkS user)
     (37 F.SilkS user)
     (38 B.Mask user hide)
@@
     (zone_45_only no)
     (trace_min 0.2)
-    (segment_width 0.1)
-    (edge_width 0.1)
     (via_size 0.8)
     (via_drill 0.4)
@@
     (uvia_min_size 0.2)
     (uvia_min_drill 0.1)
+    (edge_width 0.1)
+    (segment_width 0.1)
     (pcb_text_width 0.3)
     (pcb_text_size 1.5 1.5)
@@
     (solder_mask_min_width 0.25)
     (aux_axis_origin 0 0)
-    (visible_elements 7FFFF7FF)
+    (visible_elements 7FFFFFFF)
     (pcbplotparams
       (layerselection 0x010fc_ffffffff)
@@
     )
   )
+  (gr_text "REVISION 1 - 2019/08/16\nhttps://github.com/DutchMaker/TTL-Computer" (at 201.295 53.975) (layer B.SilkS)
+    (effects (font (size 1.5 1.5) (thickness 0.3)) (justify mirror))
+  )
+  (gr_text "↓ REGISTER D ↓" (at 153.67 242.57) (layer F.SilkS)
+    (effects (font (size 4 4) (thickness 0.7)))
+  )
+  (gr_text "↓ REGISTER C ↓" (at 93.98 242.57) (layer F.SilkS)
+    (effects (font (size 4 4) (thickness 0.7)))
+  )
   (gr_text "--------------------------------------------- DESIGNED BY RUUD VAN FALIER ---------------------------------------------" (at 201.93 65.405) (layer F.SilkS)
     (effects (font (size 2 2) (thickness 0.2)))
@@
     (effects (font (size 10 10) (thickness 1.5)))
   )
-  (gr_text "PROGRAM COUNTER" (at 105.41 435.61) (layer F.SilkS)
-    (effects (font (size 4 4) (thickness 0.7)))
-  )
-  (gr_text "INSTRUCTION REGISTER" (at 92.71 370.84) (layer F.SilkS)
-    (effects (font (size 3.5 3.3) (thickness 0.7)))
-  )
-  (gr_text CONTROLLER (at 253.746 408.813) (layer F.SilkS)
+  (gr_text "↓ PROGRAM COUNTER ↓" (at 105.41 435.61) (layer F.SilkS)
     (effects (font (size 4 4) (thickness 0.7)))
   )
-  (gr_text MEMORY (at 267.335 307.34) (layer F.SilkS)
+  (gr_text "↓ INSTRUCTION ↓" (at 92.71 370.84) (layer F.SilkS)
     (effects (font (size 4 4) (thickness 0.7)))
   )
-  (gr_text "STACK POINTER" (at 105.41 307.34) (layer F.SilkS)
+  (gr_text "↓ CONTROLLER ↓" (at 253.746 408.813) (layer F.SilkS)
     (effects (font (size 4 4) (thickness 0.7)))
   )
-  (gr_text "REGISTER D" (at 153.67 242.57) (layer F.SilkS)
+  (gr_text "↓ MEMORY ↓" (at 267.335 307.34) (layer F.SilkS)
     (effects (font (size 4 4) (thickness 0.7)))
   )
-  (gr_text "REGISTER C" (at 93.98 242.57) (layer F.SilkS)
+  (gr_text "↓ STACK POINTER ↓" (at 105.41 307.34) (layer F.SilkS)
     (effects (font (size 4 4) (thickness 0.7)))
   )
-  (gr_text "REGISTER A" (at 93.98 177.8) (layer F.SilkS)
+  (gr_text "↓ REGISTER A ↓" (at 93.98 177.8) (layer F.SilkS)
     (effects (font (size 4 4) (thickness 0.7)))
   )
-  (gr_text "REGISTER B" (at 153.67 177.8) (layer F.SilkS)
+  (gr_text "↓ REGISTER B ↓" (at 153.67 177.8) (layer F.SilkS)
     (effects (font (size 4 4) (thickness 0.7)))
   )
-  (gr_text "MEMORY ACCESS REGISTER" (at 268.605 177.8) (layer F.SilkS)
+  (gr_text "↓ MEMORY ACCESS REGISTER ↓" (at 268.605 177.8) (layer F.SilkS)
     (effects (font (size 4 4) (thickness 0.7)))
   )
-  (gr_text "FLAGS REGISTER" (at 311.15 78.74) (layer F.SilkS)
+  (gr_text "↓ FLAGS ↓" (at 311.15 78.74) (layer F.SilkS)
     (effects (font (size 4 4) (thickness 0.7)))
   )
-  (gr_text "ARITHMETIC LOGIC UNIT" (at 212.09 78.74) (layer F.SilkS)
+  (gr_text "↓ ARITHMETIC LOGIC UNIT ↓" (at 212.09 78.74) (layer F.SilkS)
     (effects (font (size 4 4) (thickness 0.7)))
   )
-  (gr_text CLOCK (at 104.14 78.74) (layer F.SilkS)
+  (gr_text "↓ CLOCK ↓" (at 104.14 78.74) (layer F.SilkS)
     (effects (font (size 4 4) (thickness 0.7)))
   )
@@
   (gr_line (start 346.075 42.545) (end 346.075 527.05) (layer Edge.Cuts) (width 0.1))
   (gr_line (start 59.69 42.545) (end 346.075 42.545) (layer Edge.Cuts) (width 0.1))
-  (gr_text "STACK\nPOINTER" (at 107.061 335.788) (layer F.SilkS)
-    (effects (font (size 6 6) (thickness 1)))
-  )
   (gr_text CLOCK (at 72.771 345.44) (layer F.SilkS)
     (effects (font (size 0.75 0.75) (thickness 0.15)) (justify left))
@@
   (gr_line (start 145.923 311.023) (end 145.923 361.823) (layer F.SilkS) (width 0.5))
   (gr_line (start 64.643 311.023) (end 64.643 361.823) (layer F.SilkS) (width 0.5))
-  (gr_text "REGISTER\nD" (at 154.305 271.145) (layer F.SilkS)
-    (effects (font (size 4 4) (thickness 0.7)))
-  )
   (gr_text D6 (at 133.7633 289.56) (layer F.SilkS)
     (effects (font (size 0.75 0.75) (thickness 0.15)) (justify left))
@@
     (effects (font (size 0.65 0.65) (thickness 0.15)) (justify left))
   )
-  (gr_text "REGISTER\nC" (at 93.345 271.145) (layer F.SilkS)
-    (effects (font (size 4 4) (thickness 0.7)))
-  )
   (gr_text D0 (at 72.8033 274.32) (layer F.SilkS)
     (effects (font (size 0.75 0.75) (thickness 0.15)) (justify left))
@@
     (effects (font (size 0.75 0.75) (thickness 0.15)) (justify left))
   )
-  (gr_text "REGISTER\nB" (at 154.305 206.375) (layer F.SilkS)
-    (effects (font (size 4 4) (thickness 0.7)))
-  )
   (gr_line (start 181.3883 233.68) (end 125.5083 233.68) (layer F.SilkS) (width 0.5))
   (gr_text D1 (at 133.7633 212.09) (layer F.SilkS)
@@
     (effects (font (size 0.75 0.75) (thickness 0.15)) (justify left))
   )
-  (gr_text "REGISTER\nA" (at 93.345 206.375) (layer F.SilkS)
-    (effects (font (size 4 4) (thickness 0.7)))
-  )
   (gr_text I7 (at 106.4583 420.37) (layer F.SilkS)
     (effects (font (size 0.75 0.75) (thickness 0.15)) (justify left))
@@
     (effects (font (size 0.75 0.75) (thickness 0.15)) (justify left))
   )
-  (gr_text "INSTRUCTION\nREGISTER" (at 93.345 386.715) (layer F.SilkS)
-    (effects (font (size 4 4) (thickness 0.7)))
-  )
   (gr_text D7 (at 72.8033 227.33) (layer F.SilkS)
     (effects (font (size 0.75 0.75) (thickness 0.15)) (justify left))
@@
   (gr_line (start 64.5483 374.65) (end 120.4283 374.65) (layer F.SilkS) (width 0.5))
   (gr_line (start 120.4283 426.72) (end 64.5483 426.72) (layer F.SilkS) (width 0.5))
-  (gr_text "PROGRAM\nCOUNTER" (at 106.045 478.79) (layer F.SilkS)
-    (effects (font (size 6 6) (thickness 1)))
-  )
   (gr_text D0 (at 73.025 497.84) (layer F.SilkS)
     (effects (font (size 0.75 0.75) (thickness 0.15)) (justify left))
@@
     (effects (font (size 0.75 0.75) (thickness 0.15)) (justify left))
   )
-  (gr_text "MEMORY ACCESS REGISTER" (at 268.605 238.76) (layer F.SilkS)
-    (effects (font (size 6 6) (thickness 1)))
-  )
   (gr_text ~PC_MAR_OUT (at 202.438 203.327) (layer F.SilkS)
     (effects (font (size 0.75 0.75) (thickness 0.15)) (justify left))
@@
   (gr_line (start 339.09 295.91) (end 194.31 295.91) (layer F.SilkS) (width 0.5))
   (gr_line (start 339.09 181.61) (end 339.09 295.91) (layer F.SilkS) (width 0.5))
-  (gr_text MEMORY (at 267.335 353.695) (layer F.SilkS)
-    (effects (font (size 6 6) (thickness 1)))
-  )
   (gr_text CLOCK (at 197.993 322.707) (layer F.SilkS)
     (effects (font (size 0.75 0.75) (thickness 0.15)) (justify left))
@@
   (gr_line (start 189.865 397.51) (end 189.865 311.15) (layer F.SilkS) (width 0.5))
   (gr_line (start 339.09 397.51) (end 189.865 397.51) (layer F.SilkS) (width 0.5))
-  (gr_text "FLAGS\nREGISTER" (at 311.404 118.618) (layer F.SilkS)
-    (effects (font (size 6 6) (thickness 0.7)))
-  )
   (gr_text Fcmp_OUT (at 333.121 150.495 90) (layer F.SilkS)
     (effects (font (size 0.75 0.75) (thickness 0.15)) (justify left))
@@
   (gr_line (start 283.464 82.423) (end 339.344 82.423) (layer F.SilkS) (width 0.5))
   (gr_line (start 283.464 158.623) (end 283.464 82.423) (layer F.SilkS) (width 0.5))
-  (gr_text CONTROLLER (at 254.635 467.995) (layer F.SilkS)
-    (effects (font (size 6 6) (thickness 1)))
-  )
   (gr_text GND (at 171.45 419.227) (layer F.SilkS)
     (effects (font (size 0.75 0.75) (thickness 0.15)) (justify left))
@@
     (effects (font (size 0.75 0.75) (thickness 0.15)) (justify left))
   )
-  (gr_text CLOCK (at 104.14 116.078) (layer F.SilkS)
-    (effects (font (size 6 6) (thickness 1)))
-  )
   (gr_line (start 64.77 82.423) (end 140.97 82.423) (layer F.SilkS) (width 0.5))
   (gr_line (start 140.97 82.423) (end 140.97 151.003) (layer F.SilkS) (width 0.5))
@@
     (effects (font (size 0.75 0.75) (thickness 0.15)) (justify left))
   )
-  (gr_text "ARITHMETIC LOGIC UNIT" (at 212.725 125.603) (layer F.SilkS)
-    (effects (font (size 6 6) (thickness 1)))
-  )
   (gr_line (start 146.05 168.783) (end 146.05 82.423) (layer F.SilkS) (width 0.5))
   (gr_line (start 278.13 82.423) (end 278.13 168.783) (layer F.SilkS) (width 0.5))
@@
   (segment (start 168.4967 447.04) (end 137.6053 447.04) (width 0.25) (layer B.Cu) (net 109))
   (segment (start 137.6053 447.04) (end 110.8083 420.243) (width 0.25) (layer B.Cu) (net 109))
-  (segment (start 73.66 163.068) (end 75.7353 163.068) (width 0.35) (layer B.Cu) (net 111))
-  (segment (start 75.7353 163.068) (end 77.9305 165.2632) (width 0.35) (layer B.Cu) (net 111))
-  (segment (start 77.9305 165.2632) (end 85.1808 165.2632) (width 0.35) (layer B.Cu) (net 111))
-  (segment (start 85.1808 165.2632) (end 88.265 162.179) (width 0.35) (layer B.Cu) (net 111))
+  (segment (start 75.66 163.068) (end 78.327 165.735) (width 0.35) (layer B.Cu) (net 111))
+  (segment (start 73.66 163.068) (end 75.66 163.068) (width 0.35) (layer B.Cu) (net 111))
+  (segment (start 84.709 165.735) (end 88.265 162.179) (width 0.35) (layer B.Cu) (net 111))
+  (segment (start 78.327 165.735) (end 84.709 165.735) (width 0.35) (layer B.Cu) (net 111))
   (segment (start 289.814 152.273) (end 289.814 155.448) (width 0.35) (layer F.Cu) (net 119))
   (segment (start 68.072 340.233) (end 67.945 340.36) (width 0.35) (layer F.Cu) (net 119))
